File: PCB_receptor/PCB_receptor.sch (KiCad schematic (older format))
At the start: 6 parts, among them J1 Screw_Terminal_01x02

Commit message: Placa do Receptor atualizada
Adicionados:
LED's indicativos
Capacitores para solucinonar defeito de fábrica da Shield Ethernet
Resistores para divisor de tensão e Pull-Up
Disposição dos componentes na placa refeito
Parts:
- removed A1: Board_Ethernet_Shield_W5100, Module:Ethernet_Shield_W5100, symbol MCU_BOARDS:Board_Ethernet_Shield_W5100
- removed J1: Screw_Terminal_01x02, TerminalBlock_Phoenix:TerminalBlock_Phoenix_MKDS-1,5-2-5.08_1x02_P5.08mm_Horizontal, symbol Connector:Screw_Terminal_01x02
- added A1: Board_Ethernet_Shield_W5100-Arduino_Mega, Module:Ethernet_Shield_W5100, symbol PCB_receptor-rescue:Board_Ethernet_Shield_W5100-Arduino_Mega
- added C1, C2: CP, Capacitor_THT:CP_Radial_D8.0mm_P5.00mm, symbol Device:CP
- added D1, D2, D3: LED, LED_THT:LED_D3.0mm, symbol Device:LED
- added J1: Barrel_Jack_MountingPin, Connector_BarrelJack:BarrelJack_Wuerth_6941xx301002, symbol Connector:Barrel_Jack_MountingPin
- added R1_4k7: R1, Resistor_THT:R_Axial_DIN0204_L3.6mm_D1.6mm_P5.08mm_Horizontal, symbol Device:R
- added R2_4k7, R5_1k1: R2, Resistor_THT:R_Axial_DIN0204_L3.6mm_D1.6mm_P5.08mm_Horizontal, symbol Device:R
- 1k1: value R -> R4_1k
- DCDC_3V1: symbol Converter_DCDC:DCDC_CHINA -> PCB_receptor-rescue:DCDC_CHINA-Converter_DCDC
- renumbered 0,5k1 to R3_0,5k1
Connections:
- net labels added: A0, A1, A2, GND_LED, RST
- no-connect marks 20 -> 18
Other:
- note added: "2 x 0,1uF\nem série"
- note added: "Cap. Shield ETH"
- note added: "Conector P4 Alimentação"
- note added: "Leds Indicativos"
- note added: "RESISTORES \nDE PULL-UP"
- note added: "Resistor Led"
- moved on the sheet: LORA_1W1, R3_0,5k1

Commit message: Atualização placa do receptor
Up
Parts:
- removed DCDC_3V1: DCDC_CHINA, Converter_DCDC:STEPDOWN_CHINA, symbol PCB_receptor-rescue:DCDC_CHINA-Converter_DCDC
- added STEPDOWN1: Converter_DCDC_STEPDOWN, Converter_DCDC:STEPDOWN_XL4005, symbol PCB_receptor-rescue:Converter_DCDC_STEPDOWN
- 1k1, R3_0,5k1: symbol Device:R -> PCB_receptor-rescue:R-Device
- C1, C2: value CP -> 0,1uF; symbol Device:CP -> PCB_receptor-rescue:CP-Device
- D1, D2, D3: symbol Device:LED -> PCB_receptor-rescue:LED-Device
- J1: symbol Connector:Barrel_Jack_MountingPin -> PCB_receptor-rescue:Barrel_Jack_MountingPin-Connector
- LORA_1W1: symbol RF_WiFi:LORA_433T30D -> PCB_receptor-rescue:LORA_433T30D-RF_WiFi
- R1: renamed from R1_4k7; value R1 -> 4K7; symbol Device:R -> PCB_receptor-rescue:R-Device
- R2: renamed from R2_4k7; value R2 -> 4K7; symbol Device:R -> PCB_receptor-rescue:R-Device
- R5: renamed from R5_1k1; value R2 -> 100; symbol Device:R -> PCB_receptor-rescue:R-Device
Connections:
- net labels added: A3
- net labels removed: A2
Other:
- moved on the sheet: R3_0,5k1
Changed lines of the file:
@@
 $EndDescr
 $Comp
-L RF_WiFi:LORA_433T30D LORA_1W1
-U 1 1 5ECF05E8
-P 6405 4040
-F 0 "LORA_1W1" H 6210 4500 50  0000 L CNN
-F 1 "LORA_433T30D" H 6140 4620 50  0000 L CNN
-F 2 "RF_WiFi:LORA_E32_433T30D" H 5885 4745 50  0000 L CNN
-F 3 "" H 6391 4076 50  0001 C CNN
-	1    6405 4040
-	1    0    0    -1
-$EndComp
-Text GLabel 6105 4340 3    50   Input ~ 0
-M0
-Text GLabel 6205 4340 3    50   Input ~ 0
-M1
-Text GLabel 6305 4340 3    50   Input ~ 0
+L PCB_receptor-rescue:GND-power #PWR05
+U 1 1 5ECF59ED
+P 7285 3555
+F 0 "#PWR05" H 7285 3305 50  0001 C CNN
+F 1 "GND" H 7290 3382 50  0000 C CNN
+F 2 "" H 7285 3555 50  0001 C CNN
+F 3 "" H 7285 3555 50  0001 C CNN
+	1    7285 3555
+	-1   0    0    1
+$EndComp
+Text GLabel 7635 4405 3    50   Input ~ 0
+3.3V_DCDC
+Text GLabel 8460 3190 0    50   Input ~ 0
 RX_LORA
-Text GLabel 6405 4340 3    50   Input ~ 0
-TX_LORA
-Text GLabel 6605 4340 3    50   Input ~ 0
-3.3V_DCDC
-$Comp
-L power:GND #PWR02
-U 1 1 5ECF37BB
-P 6705 4340
-F 0 "#PWR02" H 6705 4090 50  0001 C CNN
-F 1 "GND" H 6710 4167 50  0000 C CNN
-F 2 "" H 6705 4340 50  0001 C CNN
-F 3 "" H 6705 4340 50  0001 C CNN
-	1    6705 4340
-	1    0    0    -1
-$EndComp
-$Comp
-L PCB_receptor-rescue:DCDC_CHINA-Converter_DCDC DCDC_3V1
-U 1 1 5ECF4E65
-P 7445 4035
-F 0 "DCDC_3V1" H 7255 4840 50  0000 L CNN
-F 1 "DCDC_CHINA" H 7215 4970 50  0000 L CNN
-F 2 "Converter_DCDC:STEPDOWN_CHINA" H 6810 5100 50  0000 L CNN
-F 3 "" H 7445 4035 50  0001 C CNN
-	1    7445 4035
-	1    0    0    -1
-$EndComp
-$Comp
-L power:GND #PWR05
-U 1 1 5ECF59ED
-P 7295 3585
-F 0 "#PWR05" H 7295 3335 50  0001 C CNN
-F 1 "GND" H 7300 3412 50  0000 C CNN
-F 2 "" H 7295 3585 50  0001 C CNN
-F 3 "" H 7295 3585 50  0001 C CNN
-	1    7295 3585
-	-1   0    0    1
-$EndComp
-Text GLabel 7645 4435 3    50   Input ~ 0
-3.3V_DCDC
-Text GLabel 8335 4090 0    50   Input ~ 0
-RX_LORA
-$Comp
-L Device:R 1k1
+$Comp
+L PCB_receptor-rescue:R-Device 1k1
 U 1 1 5ED11BDF
-P 8650 4095
-F 0 "1k1" H 8720 4141 50  0001 L CNN
-F 1 "R4_1k" H 8720 4050 50  0000 L CNN
-F 2 "Resistor_THT:R_Axial_DIN0204_L3.6mm_D1.6mm_P5.08mm_Horizontal" V 8580 4095 50  0001 C CNN
-F 3 "~" H 8650 4095 50  0001 C CNN
-	1    8650 4095
+P 8775 3195
+F 0 "1k1" H 8845 3241 50  0001 L CNN
+F 1 "R4_1k" H 8845 3150 50  0000 L CNN
+F 2 "Resistor_THT:R_Axial_DIN0204_L3.6mm_D1.6mm_P5.08mm_Horizontal" V 8705 3195 50  0001 C CNN
+F 3 "~" H 8775 3195 50  0001 C CNN
+	1    8775 3195
 	0    -1   1    0
 $EndComp
 $Comp
-L power:GND #PWR0101
+L PCB_receptor-rescue:GND-power #PWR0101
 U 1 1 5ED12F2B
-P 8800 3850
-F 0 "#PWR0101" H 8800 3600 50  0001 C CNN
-F 1 "GND" H 8805 3677 50  0000 C CNN
-F 2 "" H 8800 3850 50  0001 C CNN
-F 3 "" H 8800 3850 50  0001 C CNN
-	1    8800 3850
+P 8925 2950
+F 0 "#PWR0101" H 8925 2700 50  0001 C CNN
+F 1 "GND" H 8930 2777 50  0000 C CNN
+F 2 "" H 8925 2950 50  0001 C CNN
+F 3 "" H 8925 2950 50  0001 C CNN
+	1    8925 2950
 	0    -1   1    0
 $EndComp
 $Comp
-L Device:R R3_0,5k1
+L PCB_receptor-rescue:R-Device R3_0,5k1
 U 1 1 5ECF295D
-P 8650 3850
-F 0 "R3_0,5k1" H 8720 3896 50  0000 L CNN
-F 1 "R" H 8720 3805 50  0001 L CNN
-F 2 "Resistor_THT:R_Axial_DIN0204_L3.6mm_D1.6mm_P5.08mm_Horizontal" V 8580 3850 50  0001 C CNN
-F 3 "~" H 8650 3850 50  0001 C CNN
-	1    8650 3850
+P 8775 2950
+F 0 "R3_0,5k1" H 8845 2996 50  0000 L CNN
+F 1 "R" H 8845 2905 50  0001 L CNN
+F 2 "Resistor_THT:R_Axial_DIN0204_L3.6mm_D1.6mm_P5.08mm_Horizontal" V 8705 2950 50  0001 C CNN
+F 3 "~" H 8775 2950 50  0001 C CNN
+	1    8775 2950
 	0    1    -1   0
 $EndComp
 Wire Wire Line
-	8335 4090 8500 4090
-Wire Wire Line
-	8500 4095 8500 4090
-Connection ~ 8500 4090
-Wire Wire Line
-	8500 4090 8500 3850
-NoConn ~ 6505 4340
+	8460 3190 8625 3190
+Wire Wire Line
+	8625 3195 8625 3190
+Connection ~ 8625 3190
+Wire Wire Line
+	8625 3190 8625 2950
 $Comp
 L PCB_receptor-rescue:Board_Ethernet_Shield_W5100-Arduino_Mega A1
@@
 NoConn ~ 9285 2995
 NoConn ~ 9285 3095
-NoConn ~ 9285 3195
 NoConn ~ 9285 3295
-NoConn ~ 9285 3395
-NoConn ~ 9285 3495
 NoConn ~ 9285 3595
 NoConn ~ 9285 3695
-NoConn ~ 9285 3895
-Text GLabel 9285 3795 0    50   Input ~ 0
+Text GLabel 9285 3395 0    50   Input ~ 0
 M0
-Text GLabel 9285 3995 0    50   Input ~ 0
+Text GLabel 9285 3495 0    50   Input ~ 0
 M1
-Text GLabel 9285 4195 0    50   Input ~ 0
+Text GLabel 9285 4095 0    50   Input ~ 0
 TX_LORA
-NoConn ~ 10285 3795
-$Comp
-L power:GND #PWR0102
+$Comp
+L PCB_receptor-rescue:GND-power #PWR0102
 U 1 1 5FC3B25D
 P 9785 4660
@@
 $EndComp
 $Comp
-L power:GND #PWR0103
+L PCB_receptor-rescue:GND-power #PWR0103
 U 1 1 5FC3C4B7
-P 7245 4435
-F 0 "#PWR0103" H 7245 4185 50  0001 C CNN
-F 1 "GND" H 7250 4262 50  0000 C CNN
-F 2 "" H 7245 4435 50  0001 C CNN
-F 3 "" H 7245 4435 50  0001 C CNN
-	1    7245 4435
+P 7235 4405
+F 0 "#PWR0103" H 7235 4155 50  0001 C CNN
+F 1 "GND" H 7240 4232 50  0000 C CNN
+F 2 "" H 7235 4405 50  0001 C CNN
+F 3 "" H 7235 4405 50  0001 C CNN
+	1    7235 4405
 	1    0    0    -1
 $EndComp
@@
 Text GLabel 9685 2250 1    50   Input ~ 0
 VIN
-Text GLabel 7645 3585 1    50   Input ~ 0
+Text GLabel 7635 3555 1    50   Input ~ 0
 VIN
 Text GLabel 4695 1755 3    50   Input ~ 0
 VIN
 $Comp
-L power:PWR_FLAG #FLG01
+L PCB_receptor-rescue:PWR_FLAG-power #FLG01
 U 1 1 5ECF9505
 P 4695 1755
@@
 	1    0    0    -1
 $EndComp
-Wire Wire Line
-	8800 4095 9285 4095
-$Comp
-L Device:R R1_4k7
+$Comp
+L PCB_receptor-rescue:R-Device R1
 U 1 1 5FC4CBD3
 P 5390 4135
-F 0 "R1_4k7" H 5460 4140 50  0000 L CNN
-F 1 "R1" H 5460 4090 50  0001 L CNN
+F 0 "R1" H 5475 4115 50  0000 L CNN
+F 1 "4K7" H 5450 4195 50  0000 L CNN
 F 2 "Resistor_THT:R_Axial_DIN0204_L3.6mm_D1.6mm_P5.08mm_Horizontal" V 5320 4135 50  0001 C CNN
 F 3 "~" H 5390 4135 50  0001 C CNN
@@
 $EndComp
 $Comp
-L power:GND #PWR0104
+L PCB_receptor-rescue:GND-power #PWR0104
 U 1 1 5FC51C43
 P 5390 3985
@@
 $EndComp
 $Comp
-L Device:R R2_4k7
+L PCB_receptor-rescue:R-Device R2
 U 1 1 5FC52E51
 P 5050 4140
-F 0 "R2_4k7" H 4715 4150 50  0000 L CNN
-F 1 "R2" H 5125 4085 50  0001 L CNN
+F 0 "R2" H 4865 4100 50  0000 L CNN
+F 1 "4K7" H 4835 4185 50  0000 L CNN
 F 2 "Resistor_THT:R_Axial_DIN0204_L3.6mm_D1.6mm_P5.08mm_Horizontal" V 4980 4140 50  0001 C CNN
 F 3 "~" H 5050 4140 50  0001 C CNN
@@
 $EndComp
 $Comp
-L power:GND #PWR0105
+L PCB_receptor-rescue:GND-power #PWR0105
 U 1 1 5FC53225
 P 5050 3990
@@
 RESISTORES \nDE PULL-UP
 $Comp
-L Connector:Barrel_Jack_MountingPin J1
+L PCB_receptor-rescue:Barrel_Jack_MountingPin-Connector J1
 U 1 1 5FC650E8
 P 4125 4090
@@
 VIN
 $Comp
-L power:GND #PWR0106
+L PCB_receptor-rescue:GND-power #PWR0106
 U 1 1 5FC68051
 P 4025 4390
@@
 Conector P4 Alimentação
 $Comp
-L Device:LED D1
+L PCB_receptor-rescue:LED-Device D1
 U 1 1 5FC7EEB3
 P 2455 4185
@@
 $EndComp
 $Comp
-L Device:LED D2
+L PCB_receptor-rescue:LED-Device D2
 U 1 1 5FC7F3B6
 P 2095 4185
@@
 A1
 Text GLabel 2455 4335 3    50   Input ~ 0
-A2
+A3
 Text Notes 1820 3565 0    50   ~ 0
 Leds Indicativos
@@
 A1
 $Comp
-L Device:LED D3
+L PCB_receptor-rescue:LED-Device D3
 U 1 1 5FC8532F
 P 1790 4185
@@
 Text GLabel 1790 4335 3    50   Input ~ 0
 A0
-Text GLabel 10285 3695 2    50   Input ~ 0
-A2
-$Comp
-L Device:R R5_1k1
+$Comp
+L PCB_receptor-rescue:R-Device R5
 U 1 1 5FC8A8D9
 P 1055 4175
-F 0 "R5_1k1" H 720 4185 50  0000 L CNN
-F 1 "R2" H 1130 4120 50  0001 L CNN
+F 0 "R5" H 865 4215 50  0000 L CNN
+F 1 "100" H 845 4135 50  0000 L CNN
 F 2 "Resistor_THT:R_Axial_DIN0204_L3.6mm_D1.6mm_P5.08mm_Horizontal" V 985 4175 50  0001 C CNN
 F 3 "~" H 1055 4175 50  0001 C CNN
@@
 Resistor Led
 $Comp
-L Device:CP C2
+L PCB_receptor-rescue:CP-Device C2
 U 1 1 5FC7046A
 P 3005 3995
 F 0 "C2" H 3123 4041 50  0000 L CNN
-F 1 "CP" H 3123 3950 50  0000 L CNN
+F 1 "0,1uF" H 3123 3950 50  0000 L CNN
 F 2 "Capacitor_THT:CP_Radial_D8.0mm_P5.00mm" H 3043 3845 50  0001 C CNN
 F 3 "~" H 3005 3995 50  0001 C CNN
@@
 $EndComp
 $Comp
-L power:GND #PWR01
+L PCB_receptor-rescue:GND-power #PWR01
 U 1 1 5FC8A8DF
 P 1055 4325
@@
 $EndComp
 $Comp
-L power:GND #PWR03
+L PCB_receptor-rescue:GND-power #PWR03
 U 1 1 5FC715E1
 P 3005 4445
@@
 $EndComp
 $Comp
-L Device:CP C1
+L PCB_receptor-rescue:CP-Device C1
 U 1 1 5FC6F8E3
 P 3005 4295
 F 0 "C1" H 3123 4341 50  0000 L CNN
-F 1 "CP" H 3123 4250 50  0000 L CNN
+F 1 "0,1uF" H 3123 4250 50  0000 L CNN
 F 2 "Capacitor_THT:CP_Radial_D8.0mm_P5.00mm" H 3043 4145 50  0001 C CNN
 F 3 "~" H 3005 4295 50  0001 C CNN
@@
 Text Notes 2850 4900 0    50   ~ 0
 2 x 0,1uF\nem série
+$Comp
+L PCB_receptor-rescue:LORA_433T30D-RF_WiFi LORA_1W1
+U 1 1 5ECF05E8
+P 6405 4040
+F 0 "LORA_1W1" H 6210 4500 50  0000 L CNN
+F 1 "LORA_433T30D" H 6140 4620 50  0000 L CNN
+F 2 "RF_WiFi:LORA_E32_433T30D" H 5885 4745 50  0001 L CNN
+F 3 "" H 6391 4076 50  0001 C CNN
+	1    6405 4040
+	1    0    0    -1
+$EndComp
+NoConn ~ 6505 4340
+$Comp
+L PCB_receptor-rescue:GND-power #PWR02
+U 1 1 5ECF37BB
+P 6705 4340
+F 0 "#PWR02" H 6705 4090 50  0001 C CNN
+F 1 "GND" H 6710 4167 50  0000 C CNN
+F 2 "" H 6705 4340 50  0001 C CNN
+F 3 "" H 6705 4340 50  0001 C CNN
+	1    6705 4340
+	1    0    0    -1
+$EndComp
+Text GLabel 6605 4340 3    50   Input ~ 0
+3.3V_DCDC
+Text GLabel 6405 4340 3    50   Input ~ 0
+TX_LORA
+Text GLabel 6305 4340 3    50   Input ~ 0
+RX_LORA
+Text GLabel 6205 4340 3    50   Input ~ 0
+M1
+Text GLabel 6105 4340 3    50   Input ~ 0
+M0
+$Comp
+L PCB_receptor-rescue:Converter_DCDC_STEPDOWN STEPDOWN1
+U 1 1 5FE4076C
+P 7435 4005
+F 0 "STEPDOWN1" H 7763 4121 50  0001 L CNN
+F 1 "Converter_DCDC_STEPDOWN" H 6920 4840 50  0000 L CNN
+F 2 "Converter_DCDC:STEPDOWN_XL4005" H 7763 3985 50  0001 L CNN
+F 3 "" H 7435 4005 50  0001 C CNN
+	1    7435 4005
+	1    0    0    -1
+$EndComp
+NoConn ~ 9285 4195
+NoConn ~ 9285 3795
+NoConn ~ 9285 3895
+NoConn ~ 9285 3995
+Wire Wire Line
+	8925 3195 9285 3195
+NoConn ~ 10285 3695
+Text GLabel 10285 3795 2    50   Input ~ 0
+A3
 $EndSCHEMATC
