File: PCB_transmissores/PCB_transmissores.sch (KiCad schematic (older format))
At the start: 7 parts, among them J1 Screw_Terminal_01x02

Commit message: Modificações placa transmissores
Adicionado:
Suporte de bateria
Furos de fixação
Resistores divisores de tensão
Corrigida a posição dos pinos do módulo GPS
Parts:
- added BT1: Battery_Cell, Battery:BatteryHolder_MPD_BH-18650-PC2, symbol Device:Battery_Cell
- added R1: 1k, Resistor_THT:R_Axial_DIN0207_L6.3mm_D2.5mm_P7.62mm_Horizontal, symbol Device:R
- added R2: 0,5k, Resistor_THT:R_Axial_DIN0207_L6.3mm_D2.5mm_P7.62mm_Horizontal, symbol Device:R
Connections:
- wire segments 7 -> 10
Changed lines of the file:
@@
 TX_GPS
 Text GLabel 1700 3550 3    50   Input ~ 0
-VIN
+5V_NANO
 Text GLabel 1600 3550 3    50   Input ~ 0
 RX_GPS
@@
 TX_LORA
 Text GLabel 5990 2790 0    50   Input ~ 0
-RX_GPS
-Text GLabel 5990 2890 0    50   Input ~ 0
 TX_GPS
 NoConn ~ 8660 3840
@@
 F 0 "DCDC_3V1" H 4178 3416 50  0000 L CNN
 F 1 "DCDC_CHINA" H 4178 3325 50  0000 L CNN
-F 2 "Converter_DCDC:STEPDOWN_CHINA" H 4200 3150 50  0000 L CNN
+F 2 "Converter_DCDC:STEPDOWN_CHINA" H 3210 4120 50  0000 L CNN
 F 3 "" H 3850 3300 50  0001 C CNN
 	1    3850 3300
@@
 F 0 "6M1" H 1878 3408 50  0000 L CNN
 F 1 "NEO_6M" H 1878 3317 50  0000 L CNN
-F 2 "RF_GPS:Neo-6M" H 1878 3226 50  0000 L CNN
+F 2 "RF_GPS:Neo-6M" H 1220 3700 50  0000 L CNN
 F 3 "" H 1500 3300 50  0001 C CNN
 	1    1500 3300
 	1    0    0    -1
 $EndComp
+Wire Wire Line
+	5030 2890 5150 2890
+Connection ~ 5150 2890
+Wire Wire Line
+	5150 2890 5150 3030
+$Comp
+L Device:R R1
+U 1 1 5EEE284B
+P 5300 2890
+F 0 "R1" H 5370 2936 50  0001 L CNN
+F 1 "1k" V 5323 2845 50  0000 L BNN
+F 2 "Resistor_THT:R_Axial_DIN0207_L6.3mm_D2.5mm_P7.62mm_Horizontal" V 5230 2890 50  0001 C CNN
+F 3 "~" H 5300 2890 50  0001 C CNN
+	1    5300 2890
+	0    1    1    0
+$EndComp
+$Comp
+L Device:R R2
+U 1 1 5EEE2837
+P 5300 3030
+F 0 "R2" H 5370 3076 50  0001 L CNN
+F 1 "0,5k" V 5326 2946 50  0000 L BNN
+F 2 "Resistor_THT:R_Axial_DIN0207_L6.3mm_D2.5mm_P7.62mm_Horizontal" V 5230 3030 50  0001 C CNN
+F 3 "~" H 5300 3030 50  0001 C CNN
+	1    5300 3030
+	0    1    1    0
+$EndComp
+Text GLabel 5030 2890 0    50   Input ~ 0
+RX_GPS
+$Comp
+L Device:Battery_Cell BT1
+U 1 1 5EEE89DD
+P 8000 2450
+F 0 "BT1" H 8118 2546 50  0000 L CNN
+F 1 "Battery_Cell" H 8118 2455 50  0000 L CNN
+F 2 "Battery:BatteryHolder_MPD_BH-18650-PC2" V 8000 2510 50  0001 C CNN
+F 3 "~" V 8000 2510 50  0001 C CNN
+	1    8000 2450
+	1    0    0    -1
+$EndComp
+$Comp
+L power:GND #PWR05
+U 1 1 5EEEAF42
+P 8000 2550
+F 0 "#PWR05" H 8000 2300 50  0001 C CNN
+F 1 "GND" H 8005 2377 50  0000 C CNN
+F 2 "" H 8000 2550 50  0001 C CNN
+F 3 "" H 8000 2550 50  0001 C CNN
+	1    8000 2550
+	1    0    0    -1
+$EndComp
+Text GLabel 8000 2250 1    50   Input ~ 0
+VIN
+Wire Wire Line
+	5450 2890 5990 2890
+$Comp
+L power:GND #PWR0102
+U 1 1 5EF0CBB2
+P 5450 3030
+F 0 "#PWR0102" H 5450 2780 50  0001 C CNN
+F 1 "GND" H 5455 2857 50  0000 C CNN
+F 2 "" H 5450 3030 50  0001 C CNN
+F 3 "" H 5450 3030 50  0001 C CNN
+	1    5450 3030
+	0    -1   -1   0
+$EndComp
 $EndSCHEMATC

Commit message: Subtituito StepDown por StepUp
Substituido o uso do StepDown DcDc por StepUp DcDc.
Feitas modificações em trilhas e ligações para adaptar o circuito a mudança.
Parts:
- removed DCDC_3V1: DCDC_CHINA, Converter_DCDC:STEPDOWN_CHINA, symbol Converter_DCDC:DCDC_CHINA
- added JP1, JP2: Jumper, TestPoint:Furo_Jumper, symbol Connector:TestPoint
- added R10, R7, R8, R9: 4k7, Resistor_THT:R_Axial_DIN0207_L6.3mm_D2.5mm_P7.62mm_Horizontal, symbol Device:R
- added R5: 500k, Resistor_THT:R_Axial_DIN0207_L6.3mm_D2.5mm_P7.62mm_Horizontal, symbol Device:R
- added R6: 5000k, Resistor_THT:R_Axial_DIN0207_L6.3mm_D2.5mm_P7.62mm_Horizontal, symbol Device:R
- added XL6009E11: STEPUP, Converter_DCDC:STEPUP_XL6009E1, symbol Converter_DCDC:STEPUP
- A1: symbol MCU_BOARDS:Arduino_Nano_v3.x -> PCB_transmissores-rescue:Arduino_Nano_v3.x-MCU_BOARDS
Connections:
- net labels added: 7V_STEPUP, A2, D2, D3, D6, D9
- net labels removed: 3.3V_DCDC, 5V_NANO
- wire segments 10 -> 12
- no-connect marks 18 -> 21
Other:
- note added: "Medir Tensão Bateria"
- note added: "Pull Up Resistor"

Commit message: atualização da placa dos transmissores
Up
Parts:
- removed BT1: Battery_Cell, Battery:BatteryHolder_MPD_BH-18650-PC2, symbol Device:Battery_Cell
- removed J1: Screw_Terminal_01x02, TerminalBlock_Phoenix:TerminalBlock_Phoenix_MKDS-1,5-2-5.08_1x02_P5.08mm_Horizontal, symbol Connector:Screw_Terminal_01x02
- removed JP1, JP2: Jumper, TestPoint:Furo_Jumper, symbol Connector:TestPoint
- removed LORA_1W1: LORA_433T30D, RF_WiFi:LORA_E32_433T30D, symbol RF_WiFi:LORA_433T30D
- removed XL6009E11: STEPUP, Converter_DCDC:STEPUP_XL6009E1, symbol Converter_DCDC:STEPUP
- added H1, H2: MountingHole, MountingHole:MountingHole_5.5mm, symbol Mechanical:MountingHole
- added J2: Barrel_Jack_MountingPin, Connector_BarrelJack:BarrelJack_Wuerth_6941xx301002, symbol Connector:Barrel_Jack_MountingPin
- added LORA_100mW1: LORA_433T20D, RF_WiFi:LORA_E32_433T20D, symbol RF_WiFi:LORA_433T20D
- added XL40051: STEPDOWN, Converter_DCDC:STEPDOWN_XL4005, symbol Converter_DCDC:STEPDOWN
- R5: value 500k -> 5k
- R6: value 5000k -> 36k
Connections:
- net 7V_STEPUP is gone; now on net VIN: A1.30 (VIN)
- net D9: now also LORA_100mW1.4 (TX)
- net GND: now also J2.2, LORA_100mW1.7 (GND), XL40051.1 (IN-), XL40051.3 (OUT-)
- net M0: now also LORA_100mW1.1 (M0)
- net M1: now also LORA_100mW1.2 (M1)
- net RX_LORA: now also LORA_100mW1.3 (RX)
- net VIN: now also J2.1, XL40051.2 (IN+); no longer 6M1.4 (VCC)
- net D11: now reaches A1.14 (D11)
- net D11: now also 6M1.2 (TX), R9.1
- net D12: now reaches A1.15 (D12)
- net D12: now also R1.1
- removed net D2: 6M1.2 (TX), A1.5 (D2), R9.1
- net D3: no longer names the net of A1.6 (D3)
- net D3: no longer R1.1
- new net 3,3v: 6M1.4 (VCC), LORA_100mW1.6 (VCC), XL40051.4 (OUT+)
- no-connect marks 21 -> 22
Changed lines of the file:
@@
 Text GLabel 7440 4130 3    50   Input ~ 0
 VIN
-$Comp
-L power:PWR_FLAG #FLG0102
-U 1 1 5EC6B4A8
-P 8000 4130
-F 0 "#FLG0102" H 8000 4205 50  0001 C CNN
-F 1 "PWR_FLAG" H 8000 4303 50  0000 C CNN
-F 2 "" H 8000 4130 50  0001 C CNN
-F 3 "~" H 8000 4130 50  0001 C CNN
-	1    8000 4130
-	1    0    0    -1
-$EndComp
-$Comp
-L power:GND #PWR0108
-U 1 1 5EC6B797
-P 8000 4130
-F 0 "#PWR0108" H 8000 3880 50  0001 C CNN
-F 1 "GND" V 8005 4002 50  0000 R CNN
-F 2 "" H 8000 4130 50  0001 C CNN
-F 3 "" H 8000 4130 50  0001 C CNN
-	1    8000 4130
-	-1   0    0    -1
-$EndComp
 Text GLabel 1500 3550 3    50   Input ~ 0
 TX_GPS
@@
 F 3 "" H 1400 3550 50  0001 C CNN
 	1    1400 3550
-	-1   0    0    -1
-$EndComp
-$Comp
-L Connector:Screw_Terminal_01x02 J1
-U 1 1 5EC87D36
-P 7310 2360
-F 0 "J1" H 7390 2352 50  0000 L CNN
-F 1 "Screw_Terminal_01x02" H 7390 2261 50  0000 L CNN
-F 2 "TerminalBlock_Phoenix:TerminalBlock_Phoenix_MKDS-1,5-2-5.08_1x02_P5.08mm_Horizontal" H 7310 2360 50  0001 C CNN
-F 3 "~" H 7310 2360 50  0001 C CNN
-	1    7310 2360
-	0    -1   -1   0
-$EndComp
-Text GLabel 7310 2560 3    50   Input ~ 0
-VIN
-$Comp
-L power:GND #PWR01
-U 1 1 5EC8BC4B
-P 7410 2560
-F 0 "#PWR01" H 7410 2310 50  0001 C CNN
-F 1 "GND" V 7415 2432 50  0000 R CNN
-F 2 "" H 7410 2560 50  0001 C CNN
-F 3 "" H 7410 2560 50  0001 C CNN
-	1    7410 2560
 	-1   0    0    -1
 $EndComp
@@
 	1    0    0    -1
 $EndComp
-Text GLabel 4050 2850 1    50   Input ~ 0
-VIN
-$Comp
-L power:GND #PWR04
-U 1 1 5ECACF19
-P 3650 3700
-F 0 "#PWR04" H 3650 3450 50  0001 C CNN
-F 1 "GND" H 3655 3527 50  0000 C CNN
-F 2 "" H 3650 3700 50  0001 C CNN
-F 3 "" H 3650 3700 50  0001 C CNN
-	1    3650 3700
-	1    0    0    -1
-$EndComp
-$Comp
-L RF_WiFi:LORA_433T30D LORA_1W1
-U 1 1 5ECB6750
-P 2700 3350
-F 0 "LORA_1W1" H 2505 3950 50  0000 L CNN
-F 1 "LORA_433T30D" H 2420 3845 50  0000 L CNN
-F 2 "RF_WiFi:LORA_E32_433T30D" H 2200 3750 50  0000 L CNN
-F 3 "" H 2686 3386 50  0001 C CNN
-	1    2700 3350
-	1    0    0    -1
-$EndComp
 $Comp
 L RF_GPS:NEO_6M 6M1
@@
 $EndComp
 $Comp
-L Device:Battery_Cell BT1
-U 1 1 5EEE89DD
-P 8000 2450
-F 0 "BT1" H 8118 2546 50  0000 L CNN
-F 1 "Battery_Cell" H 8118 2455 50  0000 L CNN
-F 2 "Battery:BatteryHolder_MPD_BH-18650-PC2" V 8000 2510 50  0001 C CNN
-F 3 "~" V 8000 2510 50  0001 C CNN
-	1    8000 2450
-	1    0    0    -1
-$EndComp
-$Comp
-L power:GND #PWR05
-U 1 1 5EEEAF42
-P 8000 2550
-F 0 "#PWR05" H 8000 2300 50  0001 C CNN
-F 1 "GND" H 8005 2377 50  0000 C CNN
-F 2 "" H 8000 2550 50  0001 C CNN
-F 3 "" H 8000 2550 50  0001 C CNN
-	1    8000 2550
-	1    0    0    -1
-$EndComp
-Text GLabel 8000 2250 1    50   Input ~ 0
-VIN
-$Comp
 L Device:R R6
 U 1 1 5EFC9734
 P 7640 3310
 F 0 "R6" H 7710 3356 50  0001 L CNN
-F 1 "5000k" V 7580 3190 50  0000 L BNN
+F 1 "36k" V 7580 3190 50  0000 L BNN
 F 2 "Resistor_THT:R_Axial_DIN0207_L6.3mm_D2.5mm_P7.62mm_Horizontal" V 7570 3310 50  0001 C CNN
 F 3 "~" H 7640 3310 50  0001 C CNN
@@
 P 7640 3450
 F 0 "R5" H 7710 3496 50  0001 L CNN
-F 1 "500k" V 7750 3360 50  0000 L BNN
+F 1 "5k" V 7750 3360 50  0000 L BNN
 F 2 "Resistor_THT:R_Axial_DIN0207_L6.3mm_D2.5mm_P7.62mm_Horizontal" V 7570 3450 50  0001 C CNN
 F 3 "~" H 7640 3450 50  0001 C CNN
@@
 NoConn ~ 2800 3650
 NoConn ~ 5990 3890
-NoConn ~ 5990 3790
-NoConn ~ 5990 3690
 NoConn ~ 5990 3590
 $Comp
@@
 Text GLabel 5990 3190 0    50   Input ~ 0
 D6
-Text GLabel 5990 2890 0    50   Input ~ 0
-D3
+Text GLabel 5990 3790 0    50   Input ~ 0
+D12
 Wire Wire Line
 	7490 3310 7490 3380
@@
 Wire Wire Line
 	7490 3380 7490 3450
-Text GLabel 5990 2790 0    50   Input ~ 0
-D2
+Text GLabel 5990 3690 0    50   Input ~ 0
+D11
 $Comp
 L power:GND #PWR0104
@@
 	5020 2720 5050 2720
 Text GLabel 5050 2720 2    50   Input ~ 0
-D2
+D11
 Text GLabel 5450 2890 2    50   Input ~ 0
-D3
+D12
 Text GLabel 5450 3190 2    50   Input ~ 0
 D6
@@
 Text GLabel 5430 4150 1    50   Input ~ 0
 RX_GPS
-$Comp
-L Converter_DCDC:STEPUP XL6009E11
-U 1 1 5F1DCBFD
-P 3850 3300
-F 0 "XL6009E11" H 3635 4165 50  0000 L CNN
-F 1 "STEPUP" H 3705 4265 50  0000 L CNN
-F 2 "Converter_DCDC:STEPUP_XL6009E1" H 3500 4065 50  0000 L CNN
-F 3 "" H 3850 3300 50  0001 C CNN
-	1    3850 3300
-	1    0    0    -1
-$EndComp
+NoConn ~ 6690 2190
+$Comp
+L Converter_DCDC:STEPDOWN XL40051
+U 1 1 5F35BF7D
+P 3795 3335
+F 0 "XL40051" H 4123 3451 50  0000 L CNN
+F 1 "STEPDOWN" H 4123 3360 50  0000 L CNN
+F 2 "Converter_DCDC:STEPDOWN_XL4005" H 4123 3269 50  0000 L CNN
+F 3 "" H 3795 3335 50  0001 C CNN
+	1    3795 3335
+	1    0    0    -1
+$EndComp
+Text GLabel 3995 2885 1    50   Input ~ 0
+VIN
 $Comp
 L power:GND #PWR03
-U 1 1 5ECAC6BC
-P 3700 2850
-F 0 "#PWR03" H 3700 2600 50  0001 C CNN
-F 1 "GND" H 3705 2677 50  0000 C CNN
-F 2 "" H 3700 2850 50  0001 C CNN
-F 3 "" H 3700 2850 50  0001 C CNN
-	1    3700 2850
+U 1 1 5F35C859
+P 3645 2885
+F 0 "#PWR03" H 3645 2635 50  0001 C CNN
+F 1 "GND" H 3650 2712 50  0000 C CNN
+F 2 "" H 3645 2885 50  0001 C CNN
+F 3 "" H 3645 2885 50  0001 C CNN
+	1    3645 2885
 	-1   0    0    1
 $EndComp
+Text GLabel 3995 3735 3    50   Input ~ 0
+3,3v
 Text GLabel 2900 3650 3    50   Input ~ 0
+3,3v
+Text GLabel 1700 3550 3    50   Input ~ 0
+3,3v
+Text GLabel 6390 2190 1    50   Input ~ 0
 VIN
-Text GLabel 1700 3550 3    50   Input ~ 0
+$Comp
+L Connector:Barrel_Jack_MountingPin J2
+U 1 1 5F43899E
+P 9750 4155
+F 0 "J2" H 9807 4472 50  0000 C CNN
+F 1 "Barrel_Jack_MountingPin" H 9807 4381 50  0000 C CNN
+F 2 "Connector_BarrelJack:BarrelJack_Wuerth_6941xx301002" H 9800 4115 50  0001 C CNN
+F 3 "~" H 9800 4115 50  0001 C CNN
+	1    9750 4155
+	0    1    1    0
+$EndComp
+Text GLabel 9850 4455 3    50   Input ~ 0
 VIN
-Text GLabel 4050 3700 3    50   Input ~ 0
-7V_STEPUP
-Text GLabel 6390 2190 1    50   Input ~ 0
-7V_STEPUP
-NoConn ~ 6690 2190
-$Comp
-L Connector:TestPoint JP1
-U 1 1 5F1F32C6
-P 8500 4135
-F 0 "JP1" H 8558 4253 50  0000 L CNN
-F 1 "Jumper" H 8558 4162 50  0000 L CNN
-F 2 "TestPoint:Furo_Jumper" H 8700 4135 50  0001 C CNN
-F 3 "~" H 8700 4135 50  0001 C CNN
-	1    8500 4135
-	1    0    0    -1
-$EndComp
-$Comp
-L Connector:TestPoint JP2
-U 1 1 5F1F390C
-P 8975 4130
-F 0 "JP2" H 9033 4248 50  0000 L CNN
-F 1 "Jumper" H 9033 4157 50  0000 L CNN
-F 2 "TestPoint:Furo_Jumper" H 9175 4130 50  0001 C CNN
-F 3 "~" H 9175 4130 50  0001 C CNN
-	1    8975 4130
-	1    0    0    -1
-$EndComp
-Text GLabel 8500 4135 3    50   Input ~ 0
-VIN
-Text GLabel 8975 4130 3    50   Input ~ 0
-VIN
+$Comp
+L power:GND #PWR0110
+U 1 1 5F43CE10
+P 9650 4455
+F 0 "#PWR0110" H 9650 4205 50  0001 C CNN
+F 1 "GND" V 9655 4327 50  0000 R CNN
+F 2 "" H 9650 4455 50  0001 C CNN
+F 3 "" H 9650 4455 50  0001 C CNN
+	1    9650 4455
+	-1   0    0    -1
+$EndComp
+NoConn ~ 9450 4155
+NoConn ~ 5990 2790
+NoConn ~ 5990 2890
+$Comp
+L Mechanical:MountingHole H1
+U 1 1 5F4607CD
+P 8175 2340
+F 0 "H1" H 8275 2386 50  0000 L CNN
+F 1 "MountingHole" H 8275 2295 50  0000 L CNN
+F 2 "MountingHole:MountingHole_5.5mm" H 8175 2340 50  0001 C CNN
+F 3 "~" H 8175 2340 50  0001 C CNN
+	1    8175 2340
+	1    0    0    -1
+$EndComp
+$Comp
+L Mechanical:MountingHole H2
+U 1 1 5F460A69
+P 8180 2580
+F 0 "H2" H 8280 2626 50  0000 L CNN
+F 1 "MountingHole" H 8280 2535 50  0000 L CNN
+F 2 "MountingHole:MountingHole_5.5mm" H 8180 2580 50  0001 C CNN
+F 3 "~" H 8180 2580 50  0001 C CNN
+	1    8180 2580
+	1    0    0    -1
+$EndComp
+$Comp
+L RF_WiFi:LORA_433T20D LORA_100mW1
+U 1 1 5F94CE06
+P 2700 3350
+F 0 "LORA_100mW1" H 2430 4015 50  0000 L CNN
+F 1 "LORA_433T20D" H 2420 3905 50  0000 L CNN
+F 2 "RF_WiFi:LORA_E32_433T20D" H 2180 3795 50  0000 L CNN
+F 3 "" H 2686 3386 50  0001 C CNN
+	1    2700 3350
+	1    0    0    -1
+$EndComp
+$Comp
+L power:GND #PWR0111
+U 1 1 5F95ACE7
+P 3595 3735
+F 0 "#PWR0111" H 3595 3485 50  0001 C CNN
+F 1 "GND" H 3600 3562 50  0000 C CNN
+F 2 "" H 3595 3735 50  0001 C CNN
+F 3 "" H 3595 3735 50  0001 C CNN
+	1    3595 3735
+	1    0    0    -1
+$EndComp
+$Comp
+L power:PWR_FLAG #FLG0102
+U 1 1 5F95C776
+P 8130 4135
+F 0 "#FLG0102" H 8130 4210 50  0001 C CNN
+F 1 "PWR_FLAG" H 8130 4308 50  0000 C CNN
+F 2 "" H 8130 4135 50  0001 C CNN
+F 3 "~" H 8130 4135 50  0001 C CNN
+	1    8130 4135
+	1    0    0    -1
+$EndComp
+$Comp
+L power:GND #PWR0108
+U 1 1 5F95CCA2
+P 8130 4135
+F 0 "#PWR0108" H 8130 3885 50  0001 C CNN
+F 1 "GND" H 8135 3962 50  0000 C CNN
+F 2 "" H 8130 4135 50  0001 C CNN
+F 3 "" H 8130 4135 50  0001 C CNN
+	1    8130 4135
+	1    0    0    -1
+$EndComp
 $EndSCHEMATC

Commit message: Atualização placa dos transmissores
Up
Parts:
- added D1, D2: LED, LED_THT:LED_D5.0mm, symbol Device:LED
- added R11: 100, Resistor_THT:R_Axial_DIN0207_L6.3mm_D2.5mm_P7.62mm_Horizontal, symbol Device:R
- R1, R3: value 1k -> 240
- R2, R4: value 0,5k -> 560
- R6: value 36k -> 10k
Connections:
- net A2: now also D1.2 (A); no longer R5.2, R6.2
- net GND: now also R11.2
- net A3: now reaches A1.22 (A3)
- net A3: now also D2.2 (A)
- net A7: now reaches A1.26 (A7)
- net A7: now also R5.2, R6.2
- new net R11: D1.1 (K), D2.1 (K), R11.1
- no-connect marks 22 -> 21
Other:
- note added: "LEDS indicativos"
- moved on the sheet: 6M1, A1, H1, H2, J2, LORA_100mW1, XL40051
